File: v.1 display_leds/shield_display.kicad_pcb (KiCad board)
At the start: 2 copper layers, 65 x 56.5 mm, 55 parts, among them P1 CONN_02X20, Q1 MMBT3906, Q2 MMBT3906, Q3 MMBT3906, Q4 MMBT3906, SW1 PTS645SM43SMTR92 LFS, SW10 EG1218, SW2 PTS645SM43SMTR92 LFS, SW3 EG1218, SW4 EG1218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

Commit message: ok
Other:
- rule via_min_size: 0.4 -> 0.6
Changed lines of the file:
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@@
   (layers
     (0 F.Cu signal)
-    (31 B.Cu signal)
+    (31 B.Cu signal hide)
     (32 B.Adhes user hide)
     (33 F.Adhes user hide)
@@
     (36 B.SilkS user hide)
     (37 F.SilkS user)
-    (38 B.Mask user hide)
-    (39 F.Mask user hide)
+    (38 B.Mask user)
+    (39 F.Mask user)
     (40 Dwgs.User user hide)
     (41 Cmts.User user hide)
@@
     (user_trace_width 0.5)
     (trace_clearance 0.2)
-    (zone_clearance 0.5)
+    (zone_clearance 0.4)
     (zone_45_only no)
     (trace_min 0.01)
     (via_size 0.6)
     (via_drill 0.4)
-    (via_min_size 0.4)
+    (via_min_size 0.6)
     (via_min_drill 0.3)
     (uvia_size 0.3)
@@
     (visible_elements 7FFFFFFF)
     (pcbplotparams
-      (layerselection 0x01020_80000001)
+      (layerselection 0x010f0_ffffffff)
       (usegerberextensions false)
       (usegerberattributes false)
@@
   (segment (start 143.891 74.0784) (end 143.891 69.7484) (width 0.2) (layer F.Cu) (net 55) (status 10))
   (zone (net 1) (net_name GND) (layer F.Cu) (hatch edge 0.508)
-    (connect_pads (clearance 0.5))
-    (min_thickness 0.254)
-    (fill yes (arc_segments 16) (thermal_gap 0.508) (thermal_bridge_width 0.508))
+    (connect_pads yes (clearance 0.4))
+    (min_thickness 0.4)
+    (fill yes (arc_segments 16) (thermal_gap 2) (thermal_bridge_width 2))
     (polygon
       (pts
@@
   )
   (zone (net 1) (net_name GND) (layer B.Cu) (hatch edge 0.508)
-    (connect_pads (clearance 0.5))
-    (min_thickness 0.254)
-    (fill yes (arc_segments 16) (thermal_gap 0.508) (thermal_bridge_width 0.508))
+    (connect_pads yes (clearance 0.6))
+    (min_thickness 0.6)
+    (fill yes (arc_segments 16) (thermal_gap 2) (thermal_bridge_width 2))
     (polygon
       (pts
